Commit message: Add aloha (single) robot model

File: jrl/urdfs/aloha/gazebo_dual_vx300s_formatted.urdf (robot description, URDF)
Before this commit: robot dual_vx300s, 35 links, 34 joints
Links:
- removed link puppet_right/base_link
- removed link puppet_right/ee_arm_link
- removed link puppet_right/ee_gripper_link
- removed link puppet_right/fingers_link
- removed link puppet_right/gripper_bar_link
- removed link puppet_right/gripper_link
- removed link puppet_right/gripper_prop_link
- removed link puppet_right/left_finger_link
- removed link puppet_right/lower_forearm_link
- removed link puppet_right/middle2_finger_link
- removed link puppet_right/middle_finger_link
- removed link puppet_right/right_finger_link
- removed link puppet_right/shoulder_link
- removed link puppet_right/upper_arm_link
- removed link puppet_right/upper_forearm_link
- removed link puppet_right/wrist_link
- link puppet_left/base_link: geometry collision mesh filename=urdfs/aloha/meshes/collision/vx300s_1_base.stl scale=0.001 0.001 0.001; visual mesh filename=urdfs/aloha/meshes/visual/vx300s_1_base.stl scale=0.001 0.001 0.001
- link puppet_left/gripper_bar_link: geometry collision mesh filename=urdfs/aloha/meshes/collision/vx300s_9_gripper_bar.stl scale=0.001 0.001 0.001; visual mesh filename=urdfs/aloha/meshes/visual/vx300s_9_gripper_bar.stl scale=0.001 0.001 0.001
- link puppet_left/gripper_link: geometry collision mesh filename=urdfs/aloha/meshes/collision/vx300s_7_gripper.stl scale=0.001 0.001 0.001; visual mesh filename=urdfs/aloha/meshes/visual/vx300s_7_gripper.stl scale=0.001 0.001 0.001
- link puppet_left/gripper_prop_link: geometry collision mesh filename=urdfs/aloha/meshes/collision/vx300s_8_gripper_prop.stl scale=0.001 0.001 0.001; visual mesh filename=urdfs/aloha/meshes/visual/vx300s_8_gripper_prop.stl scale=0.001 0.001 0.001
- link puppet_left/left_finger_link: geometry collision mesh filename=urdfs/aloha/meshes/collision/vx300s_10_gripper_finger.stl scale=0.001 0.001 0.001; visual mesh filename=urdfs/aloha/meshes/visual/vx300s_10_gripper_finger.stl scale=0.001 0.001 0.001
- link puppet_left/lower_forearm_link: geometry collision mesh filename=urdfs/aloha/meshes/collision/vx300s_5_lower_forearm.stl scale=0.001 0.001 0.001; visual mesh filename=urdfs/aloha/meshes/visual/vx300s_5_lower_forearm.stl scale=0.001 0.001 0.001
- link puppet_left/middle2_finger_link: geometry collision mesh filename=urdfs/aloha/meshes/collision/vx300s_10_gripper_finger.stl scale=0.001 0.001 0.001; visual mesh filename=urdfs/aloha/meshes/visual/vx300s_10_gripper_finger.stl scale=0.001 0.001 0.001
- link puppet_left/middle_finger_link: geometry collision mesh filename=urdfs/aloha/meshes/collision/vx300s_10_gripper_finger.stl scale=0.001 0.001 0.001; visual mesh filename=urdfs/aloha/meshes/visual/vx300s_10_gripper_finger.stl scale=0.001 0.001 0.001
- link puppet_left/right_finger_link: geometry collision mesh filename=urdfs/aloha/meshes/collision/vx300s_10_gripper_finger.stl scale=0.001 0.001 0.001; visual mesh filename=urdfs/aloha/meshes/visual/vx300s_10_gripper_finger.stl scale=0.001 0.001 0.001
- link puppet_left/shoulder_link: geometry collision mesh filename=urdfs/aloha/meshes/collision/vx300s_2_shoulder.stl scale=0.001 0.001 0.001; visual mesh filename=urdfs/aloha/meshes/visual/vx300s_2_shoulder.stl scale=0.001 0.001 0.001
- link puppet_left/upper_arm_link: geometry collision mesh filename=urdfs/aloha/meshes/collision/vx300s_3_upper_arm.stl scale=0.001 0.001 0.001; visual mesh filename=urdfs/aloha/meshes/visual/vx300s_3_upper_arm.stl scale=0.001 0.001 0.001
- link puppet_left/upper_forearm_link: geometry collision mesh filename=urdfs/aloha/meshes/collision/vx300s_4_upper_forearm.stl scale=0.001 0.001 0.001; visual mesh filename=urdfs/aloha/meshes/visual/vx300s_4_upper_forearm.stl scale=0.001 0.001 0.001
- link puppet_left/wrist_link: geometry collision mesh filename=urdfs/aloha/meshes/collision/vx300s_6_wrist.stl scale=0.001 0.001 0.001; visual mesh filename=urdfs/aloha/meshes/visual/vx300s_6_wrist.stl scale=0.001 0.001 0.001
Joints:
- removed joint puppet_right/ee_arm
- removed joint puppet_right/ee_bar
- removed joint puppet_right/ee_gripper
- removed joint puppet_right/elbow
- removed joint puppet_right/forearm_roll
- removed joint puppet_right/gripper
- removed joint puppet_right/gripper_bar
- removed joint puppet_right/left_finger
- removed joint puppet_right/middle2_finger
- removed joint puppet_right/middle_finger
- removed joint puppet_right/right_finger
- removed joint puppet_right/shoulder
- removed joint puppet_right/waist
- removed joint puppet_right/wrist_angle
- removed joint puppet_right/wrist_rotate
- removed joint right_base
- joint camera_frame_joint: origin xyz=0.0, 0.0, 0.55 rpy=3.14159 0 0 -> xyz=0.0 0.0 0.55 rpy=3.14159 0 0
- joint left_base: origin xyz=-0.469 0 0 rpy=0 0 0 -> xyz=0 0 0 rpy=0 0 0

Commit message: Remove unused gripper finger joints and links from aloha single arm URDF

File: jrl/urdfs/aloha/gazebo_dual_vx300s_formatted.urdf (robot description, URDF)
Before this commit: robot dual_vx300s, 19 links, 18 joints
Links:
- removed link puppet_left/left_finger_link
- removed link puppet_left/middle2_finger_link
- removed link puppet_left/middle_finger_link
- removed link puppet_left/right_finger_link
Joints:
- removed joint puppet_left/left_finger
- removed joint puppet_left/middle2_finger
- removed joint puppet_left/middle_finger
- removed joint puppet_left/right_finger
